File: switch_matrix.kicad_sch (KiCad schematic)
At the start: 136 parts, among them SW10 SW_z, SW11 SW_super, SW12 SW_2, SW13 SW_w, SW14 SW_s, SW15 SW_x, SW16 SW_alt, SW17 SW_3, SW18 SW_e, SW19 SW_d, SW2 SW_`, SW20 SW_c, SW21 SW_m_left, SW22 SW_4, SW23 SW_r, SW24 SW_f, SW25 SW_v, SW26 SW_m_middle, SW27 SW_5, SW28 SW_t, SW29 SW_g, SW3 SW_tab, SW30 SW_b, SW31 SW_space, SW32 SW_6, SW33 SW_y, SW34 SW_h, SW35 SW_n, SW36 SW_m_right, SW37 SW_7, SW38 SW_u, SW39 SW_j, SW4 SW_caps, SW40 SW_m, SW41 SW_8, SW42 SW_i, SW43 SW_k, SW44 SW_,, SW45 SW_r_ctrl, SW46 SW_9, SW47 SW_o, SW48 SW_l, SW49 SW_., SW5 SW_shift, SW50 SW_fn1, SW51 SW_0, SW52 SW_p, SW53 SW_;, SW54 SW_/, SW55 SW_fn2, SW56 SW_-, SW57 SW_[, SW58 SW_', SW59 SW_r_shift, SW6 SW_ctrl, SW60 SW_left, SW61 SW_+, SW62 SW_], SW63 SW_enter, SW64 SW_up, SW65 SW_down, SW66 SW_back, SW67 SW_\, SW68 SW_esc, SW69 SW_right, SW7 SW_1, SW8 SW_q, SW9 SW_a

Commit message: Draft
Parts:
- removed D56: D, Diode_THT:D_DO-35_SOD27_P7.62mm_Horizontal, symbol Device:D
- removed SW55: SW_fn2, Switch_Keyboard_Hotswap_Kailh:SW_Hotswap_Kailh_MX_1.00u, symbol Switch:SW_SPST
- SW67: footprint Switch_Keyboard_Hotswap_Kailh:SW_Hotswap_Kailh_MX_1.00u -> Switch_Keyboard_Hotswap_Kailh:SW_Hotswap_Kailh_MX_1.50u
Changed lines of the file:
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@@
 (kicad_sch (version 20211123) (generator eeschema)
   (paper "A4")
-  (junction (at 207.01 140.97) (diameter 0) (color 0 0 0 0)
-  )
   (junction (at 69.85 69.85) (diameter 0) (color 0 0 0 0)
   )
@@
   (junction (at 85.09 123.19) (diameter 0) (color 0 0 0 0)
   )
-  (junction (at 217.17 115.57) (diameter 0) (color 0 0 0 0)
-  )
   (junction (at 130.81 140.97) (diameter 0) (color 0 0 0 0)
   )
@@
     (stroke (width 0) (type default) (color 0 0 0 0))
   )
-  (wire (pts (xy 207.01 140.97) (xy 222.25 140.97))
-    (stroke (width 0) (type default) (color 0 0 0 0))
-  )
   (wire (pts (xy 44.45 140.97) (xy 54.61 140.97))
     (stroke (width 0) (type default) (color 0 0 0 0))
@@
     (stroke (width 0) (type default) (color 0 0 0 0))
   )
-  (wire (pts (xy 191.77 140.97) (xy 207.01 140.97))
+  (wire (pts (xy 191.77 140.97) (xy 222.25 140.97))
     (stroke (width 0) (type default) (color 0 0 0 0))
   )
@@
   )
   (wire (pts (xy 201.93 62.23) (xy 201.93 80.01))
-    (stroke (width 0) (type default) (color 0 0 0 0))
-  )
-  (wire (pts (xy 217.17 115.57) (xy 217.17 133.35))
     (stroke (width 0) (type default) (color 0 0 0 0))
   )
@@
     (pin "2")
   )
-  (symbol (lib_id "Device:D") (at 207.01 137.16 90) (unit 1)
-    (in_bom yes) (on_board yes) (fields_autoplaced)
-    (property "Reference" "D56" (id 0) (at 209.55 135.8899 90)
-      (effects (font (size 1.27 1.27)) (justify right))
-    )
-    (property "Value" "D" (id 1) (at 209.55 138.4299 90)
-      (effects (font (size 1.27 1.27)) (justify right))
-    )
-    (property "Footprint" "Diode_THT:D_DO-35_SOD27_P7.62mm_Horizontal" (id 2) (at 207.01 137.16 0)
-      (effects (font (size 1.27 1.27)) hide)
-    )
-    (property "Datasheet" "~" (id 3) (at 207.01 137.16 0)
-      (effects (font (size 1.27 1.27)) hide)
-    )
-    (pin "1")
-    (pin "2")
-  )
   (symbol (lib_id "Device:D") (at 85.09 101.6 90) (unit 1)
     (in_bom yes) (on_board yes) (fields_autoplaced)
@@
     (pin "2")
   )
-  (symbol (lib_id "Switch:SW_SPST") (at 212.09 133.35 0) (unit 1)
-    (in_bom yes) (on_board yes) (fields_autoplaced)
-    (property "Reference" "SW55" (id 0) (at 212.09 127 0))
-    (property "Value" "SW_fn2" (id 1) (at 212.09 129.54 0))
-    (property "Footprint" "Switch_Keyboard_Hotswap_Kailh:SW_Hotswap_Kailh_MX_1.00u" (id 2) (at 212.09 133.35 0)
-      (effects (font (size 1.27 1.27)) hide)
-    )
-    (property "Datasheet" "~" (id 3) (at 212.09 133.35 0)
-      (effects (font (size 1.27 1.27)) hide)
-    )
-    (pin "1")
-    (pin "2")
-  )
   (symbol (lib_id "Switch:SW_SPST") (at 181.61 62.23 0) (unit 1)
     (in_bom yes) (on_board yes) (fields_autoplaced)
@@
     (property "Reference" "SW67" (id 0) (at 257.81 73.66 0))
     (property "Value" "SW_\\" (id 1) (at 257.81 76.2 0))
-    (property "Footprint" "Switch_Keyboard_Hotswap_Kailh:SW_Hotswap_Kailh_MX_1.00u" (id 2) (at 257.81 80.01 0)
-      (effects (font (size 1.27 1.27)) hide)
-    )
+    (property "Footprint" "Switch_Keyboard_Hotswap_Kailh:SW_Hotswap_Kailh_MX_1.50u" (id 2) (at 257.81 80.01 0)
+      (effects (font (size 1.27 1.27)) hide)
+    )

Commit message: V1, before a major change
Parts:
- SW45: value SW_r_ctrl -> SW_fn1
- SW50: value SW_fn1 -> SW_fn2
Other:
- title: (none) -> Switch Matrix
Changed lines of the file:
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@@
 (kicad_sch (version 20211123) (generator eeschema)
   (paper "A4")
+  (title_block
+    (title "Switch Matrix")
+    (comment 1 "CC BY-SA 2.0")
+  )
   (junction (at 69.85 69.85) (diameter 0) (color 0 0 0 0)
   )
@@
     (in_bom yes) (on_board yes) (fields_autoplaced)
     (property "Reference" "SW50" (id 0) (at 196.85 127 0))
-    (property "Value" "SW_fn1" (id 1) (at 196.85 129.54 0))
+    (property "Value" "SW_fn2" (id 1) (at 196.85 129.54 0))
     (property "Footprint" "Switch_Keyboard_Hotswap_Kailh:SW_Hotswap_Kailh_MX_1.00u" (id 2) (at 196.85 133.35 0)
       (effects (font (size 1.27 1.27)) hide)
@@
     (in_bom yes) (on_board yes) (fields_autoplaced)
     (property "Reference" "SW45" (id 0) (at 181.61 127 0))
-    (property "Value" "SW_r_ctrl" (id 1) (at 181.61 129.54 0))
+    (property "Value" "SW_fn1" (id 1) (at 181.61 129.54 0))
     (property "Footprint" "Switch_Keyboard_Hotswap_Kailh:SW_Hotswap_Kailh_MX_1.00u" (id 2) (at 181.61 133.35 0)
       (effects (font (size 1.27 1.27)) hide)

Commit message: New version
Parts:
- added D56: D, Diode_THT:D_DO-35_SOD27_P7.62mm_Horizontal, symbol Device:D
- added SW55: SW_ins, Switch_Keyboard_Hotswap_Kailh:SW_Hotswap_Kailh_MX_1.00u, symbol Switch:SW_SPST
- SW26: value SW_m_middle -> SW_del
- SW59: footprint Switch_Keyboard_Hotswap_Kailh:SW_Hotswap_Kailh_MX_1.75u -> Switch_Keyboard_Hotswap_Kailh:SW_Hotswap_Kailh_MX_2.75u
- SW64: value SW_up -> SW_down
- SW65: value SW_down -> SW_up
Connections:
- net C10: now also SW64.2 (B)
- net C11: now also SW65.2 (B); no longer SW60.2 (B)
- net C12: now also SW69.2 (B), SW55.2 (B); no longer SW64.2 (B), SW65.2 (B)
- net C13: now also SW26.2 (B); no longer SW69.2 (B)
- net C4: no longer SW26.2 (B)
- net C7: now also SW45.2 (B)
- net C8: now also SW50.2 (B); no longer SW45.2 (B)
- net C9: now also SW60.2 (B); no longer SW50.2 (B)
- net R2: no longer D69.1 (K)
- net R3: now also D69.1 (K), D56.1 (K); no longer D65.1 (K)
- net R4: now also D65.1 (K)
- new net: D56.2 (A), SW55.1 (A)
Other:
- note added: "Joystick Switch"
- note added: "Rotary Encoder Switch"
- moved on the sheet: D46, D51, D61, D65, D66, D69, D70, SW45, SW50, SW60, SW64, SW65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

Commit message: Updated edge cut layer
Connections:
- net C0: now also SW26.2 (B), SW55.2 (B), SW68.2 (B); no longer SW2.2 (B), SW3.2 (B), SW4.2 (B), SW5.2 (B)
- net C1: now also SW2.2 (B), SW3.2 (B), SW4.2 (B), SW5.2 (B); no longer SW10.2 (B), SW7.2 (B), SW8.2 (B), SW9.2 (B)
- net C10: now also SW46.2 (B), SW47.2 (B), SW48.2 (B), SW49.2 (B); no longer SW51.2 (B), SW52.2 (B), SW53.2 (B), SW54.2 (B)
- net C11: now also SW51.2 (B), SW52.2 (B), SW53.2 (B), SW54.2 (B); no longer SW56.2 (B), SW57.2 (B), SW58.2 (B), SW59.2 (B)
- net C12: now also SW56.2 (B), SW57.2 (B), SW58.2 (B), SW59.2 (B); no longer SW55.2 (B), SW61.2 (B), SW62.2 (B), SW63.2 (B)
- net C13: now also SW61.2 (B), SW62.2 (B), SW63.2 (B); no longer SW26.2 (B), SW68.2 (B)
- net C2: now also SW10.2 (B), SW7.2 (B), SW8.2 (B), SW9.2 (B); no longer SW12.2 (B), SW13.2 (B), SW14.2 (B), SW15.2 (B)
- net C3: now also SW12.2 (B), SW13.2 (B), SW14.2 (B), SW15.2 (B); no longer SW17.2 (B), SW18.2 (B), SW19.2 (B), SW20.2 (B)
- net C4: now also SW17.2 (B), SW18.2 (B), SW19.2 (B), SW20.2 (B); no longer SW22.2 (B), SW23.2 (B), SW24.2 (B), SW25.2 (B)
- net C5: now also SW22.2 (B), SW23.2 (B), SW24.2 (B), SW25.2 (B); no longer SW27.2 (B), SW28.2 (B), SW29.2 (B), SW30.2 (B)
- net C6: now also SW27.2 (B), SW28.2 (B), SW29.2 (B), SW30.2 (B); no longer SW32.2 (B), SW33.2 (B), SW34.2 (B), SW35.2 (B)
- net C7: now also SW32.2 (B), SW33.2 (B), SW34.2 (B), SW35.2 (B); no longer SW37.2 (B), SW38.2 (B), SW39.2 (B), SW40.2 (B)
- net C8: now also SW37.2 (B), SW38.2 (B), SW39.2 (B), SW40.2 (B); no longer SW41.2 (B), SW42.2 (B), SW43.2 (B), SW44.2 (B)
- net C9: now also SW41.2 (B), SW42.2 (B), SW43.2 (B), SW44.2 (B); no longer SW46.2 (B), SW47.2 (B), SW48.2 (B), SW49.2 (B)
- net R0: no longer D67.1 (K)
- net R1: now also D67.1 (K), D69.1 (K); no longer D63.1 (K), D68.1 (K)
- net R2: now also D27.1 (K), D63.1 (K); no longer D64.1 (K)
- net R3: now also D68.1 (K); no longer D69.1 (K)
- net R4: now also D64.1 (K); no longer D27.1 (K)
Other:
- moved on the sheet: D10, D11, D13, D14, D15, D16, D18, D19, D20, D21, D23, D24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
