File: PCB/pico_keyboard_v1.kicad_sch (KiCad schematic)
At the start: 15 parts, among them J1 Conn_01x04_12864, J2 Conn_01x03_Female, J3 Conn_01x03_Female, SW1 RotaryEncoder_Switch, U1 COM-09032, U2 Pico

Commit message: Fixed the RC filter for rotary encoder
Connections:
- net +3V3: now also R1.2, R2.2
- net +5V: no longer R1.2, R2.2
- net GND: now also C1.1, C2.2; no longer C1.2, C2.1
- net GPIO19: now also C1.2; no longer C1.1, R1.1
- net GPIO22: now also C2.1; no longer C2.2, R2.1
- net at R4.1, SW1.B: now also R2.1
- net at R3.1, SW1.A: now also R1.1
Other:
- moved on the sheet: C1, C2, R3, R4

Commit message: Started working on v0.5
Parts:
- removed U1: COM-09032, COM-09032:XDCR_COM-09032, symbol COM-09032:COM-09032
- added U1: RKJXV1224, RKJXV1224:RKJXV122400R, symbol RKJXV1224:RKJXV1224
- renumbered J3 to J2, J2 to J3, R5 to R1, R1 to R2, R2 to R3, R3 to R4, R4 to R5
Connections:
- net +3V3: now also U1.A11 (V+), U1.B11 (H+)
- net C12: now also U2.16 (GPIO12); no longer U2.17 (GPIO13)
- net C13: now also U2.17 (GPIO13); no longer U2.16 (GPIO12)
- net C5: now also U1.B1 (SEL-)
- net GND: now also U1.A13 (V-), U1.B13 (H-)
- net GPIO16: no longer D1.1 (K)
- net GPIO17: now also D1.1 (K)
- net GPIO27: now also U1.A12 (V)
- net GPIO28: now also U1.B12 (H)
- net at D1.2 (A): now also U1.A1 (SEL+)
- no-connect marks 5 -> 4
Other:
- moved on the sheet: D1

Commit message: Use both types of joystick
Parts:
- U1: footprint RKJXV1224:RKJXV122400R -> RKJXV1224:RKJXV122400R_COM09032
Connections:
- net C5: now also U1.D1 (SEL-); no longer U1.B1 (SEL-)
- net at D1.2 (A): now also U1.C1 (SEL+); no longer U1.A1 (SEL+)
Changed lines of the file:
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@@
     (property "Reference" "U1" (id 0) (at 62.3208 97.9424 0))
     (property "Value" "RKJXV1224" (id 1) (at 62.3208 100.4824 0))
-    (property "Footprint" "RKJXV1224:RKJXV122400R" (id 2) (at 62.2808 115.824 0)
+    (property "Footprint" "RKJXV1224:RKJXV122400R_COM09032" (id 2) (at 62.2808 115.824 0)
       (effects (font (size 1.27 1.27)) hide)
     )
@@
       (effects (font (size 1.27 1.27)) hide)
     )
-    (pin "A1")
     (pin "A11")
     (pin "A12")
     (pin "A13")
-    (pin "B1")
     (pin "B11")
     (pin "B12")
     (pin "B13")
+    (pin "C1")
+    (pin "D1")
   )
   (symbol (lib_id "power:+3.3V") (at 245.618 61.722 0) (unit 1)
@@
       (reference "D25") (unit 1) (value "D") (footprint "Diode_THT:D_DO-35_SOD27_P7.62mm_Horizontal")
     )
-    (path "/93eb0ca5-32f0-4914-ab02-ab34a84786ac/13828d37-1d60-434b-aca8-e63c25b6f448"
-      (reference "D26") (unit 1) (value "D") (footprint "Diode_THT:D_DO-35_SOD27_P7.62mm_Horizontal")
-    )
     (path "/93eb0ca5-32f0-4914-ab02-ab34a84786ac/c7739ee3-0359-4276-854b-62866e34bdb0"
       (reference "D27") (unit 1) (value "D") (footprint "Diode_THT:D_DO-35_SOD27_P7.62mm_Horizontal")
@@
       (reference "D39") (unit 1) (value "D") (footprint "Diode_THT:D_DO-35_SOD27_P7.62mm_Horizontal")
     )
-    (path "/93eb0ca5-32f0-4914-ab02-ab34a84786ac/e1993245-6a37-4b18-b14e-e01ac6d9b933"
-      (reference "D40") (unit 1) (value "D") (footprint "Diode_THT:D_DO-35_SOD27_P7.62mm_Horizontal")
-    )
     (path "/93eb0ca5-32f0-4914-ab02-ab34a84786ac/26039e68-7592-4888-8dea-472cf9d4a587"
       (reference "D41") (unit 1) (value "D") (footprint "Diode_THT:D_DO-35_SOD27_P7.62mm_Horizontal")
@@
       (reference "SW24") (unit 1) (value "SW_c") (footprint "Switch_Keyboard_Hotswap_Kailh:SW_Hotswap_Kailh_MX_1.00u")
     )
-    (path "/93eb0ca5-32f0-4914-ab02-ab34a84786ac/558aaf54-eb25-4a6d-a95d-d4bfda2e0042"
-      (reference "SW25") (unit 1) (value "SW_m_left") (footprint "Switch_Keyboard_Hotswap_Kailh:SW_Hotswap_Kailh_MX_1.00u")
-    )
     (path "/93eb0ca5-32f0-4914-ab02-ab34a84786ac/27fa72d0-710b-494f-b0a1-a76b0e9fdbf0"
       (reference "SW26") (unit 1) (value "SW_4") (footprint "Switch_Keyboard_Hotswap_Kailh:SW_Hotswap_Kailh_MX_1.00u")
@@
       (reference "SW38") (unit 1) (value "SW_n") (footprint "Switch_Keyboard_Hotswap_Kailh:SW_Hotswap_Kailh_MX_1.00u")
     )
-    (path "/93eb0ca5-32f0-4914-ab02-ab34a84786ac/4c7deccd-ec76-4eb5-9a28-9ad669414d94"
-      (reference "SW39") (unit 1) (value "SW_m_right") (footprint "Switch_Keyboard_Hotswap_Kailh:SW_Hotswap_Kailh_MX_1.00u")
-    )
     (path "/93eb0ca5-32f0-4914-ab02-ab34a84786ac/eba617b8-e217-4b0d-8a8e-2e7e77b01c04"
       (reference "SW40") (unit 1) (value "SW_7") (footprint "Switch_Keyboard_Hotswap_Kailh:SW_Hotswap_Kailh_MX_1.00u")
@@
     )
     (path "/b1fdc5f7-c90b-4888-9648-3bc1aa991ff5"
-      (reference "U1") (unit 1) (value "RKJXV1224") (footprint "RKJXV1224:RKJXV122400R")
+      (reference "U1") (unit 1) (value "RKJXV1224") (footprint "RKJXV1224:RKJXV122400R_COM09032")
     )
     (path "/a7a0813e-659b-4420-880d-3ea9fb1c80b1"
