File: PCB/switch_matrix.kicad_sch (KiCad schematic)
At the start: 136 parts, among them SW10 SW_z, SW11 SW_super, SW12 SW_2, SW13 SW_w, SW14 SW_s, SW15 SW_x, SW16 SW_alt, SW17 SW_3, SW18 SW_e, SW19 SW_d, SW2 SW_`, SW20 SW_c, SW21 SW_m_left, SW22 SW_4, SW23 SW_r, SW24 SW_f, SW25 SW_v, SW26 SW_del, SW27 SW_5, SW28 SW_t, SW29 SW_g, SW3 SW_tab, SW30 SW_b, SW31 SW_space, SW32 SW_6, SW33 SW_y, SW34 SW_h, SW35 SW_n, SW36 SW_m_right, SW37 SW_7, SW38 SW_u, SW39 SW_j, SW4 SW_caps, SW40 SW_m, SW41 SW_8, SW42 SW_i, SW43 SW_k, SW44 SW_,, SW45 SW_fn1, SW46 SW_9, SW47 SW_o, SW48 SW_l, SW49 SW_., SW5 SW_shift, SW50 SW_fn2, SW51 SW_0, SW52 SW_p, SW53 SW_;, SW54 SW_/, SW55 SW_ins, SW56 SW_-, SW57 SW_[, SW58 SW_', SW59 SW_r_shift, SW6 SW_ctrl, SW60 SW_left, SW61 SW_+, SW62 SW_], SW63 SW_enter, SW64 SW_down, SW65 SW_up, SW66 SW_back, SW67 SW_\, SW68 SW_esc, SW69 SW_right, SW7 SW_1, SW8 SW_q, SW9 SW_a

Commit message: Started working on v0.5
Parts:
- renumbered D6 to D10, D7 to D11, D8 to D12, D9 to D13, D10 to D14, D11 to D15, D12 to D16, D13 to D17, D14 to D18, D15 to D19, D16 to D20, D17 to D21, D18 to D22, D19 to D23, D20 to D24, D21 to D25, D22 to D26, D23 to D27, D24 to D28, D25 to D29, D69 to D3, D26 to D30, D28 to D31, D29 to D32, D30 to D33, D31 to D34, D32 to D35, D33 to D36, D34 to D37, D35 to D38, D36 to D39, D27 to D4, D37 to D40, D38 to D41, D39 to D42, D40 to D43, D41 to D44, D51 to D45, D42 to D46, D43 to D47, D44 to D48, D45 to D49, D56 to D5, D61 to D50, D47 to D51, D48 to D52, D49 to D53, D50 to D54, D65 to D55, D52 to D56, D53 to D57, D54 to D58, D55 to D59, D46 to D6, D66 to D60, D57 to D61, D58 to D62, D59 to D63, D60 to D64, D70 to D65, D62 to D66, D63 to D68, D68 to D69, D3 to D7, D64 to D70, D4 to D8, D5 to D9, SW6 to SW10, SW7 to SW11, SW8 to SW12, SW9 to SW13, SW10 to SW14, SW11 to SW15, SW12 to SW16, SW13 to SW17, SW14 to SW18, SW15 to SW19, SW68 to SW2, SW16 to SW20, SW17 to SW21, SW18 to SW22, SW19 to SW23, SW20 to SW24, SW21 to SW25, SW22 to SW26, SW23 to SW27, SW24 to SW28, SW25 to SW29, SW26 to SW3, SW27 to SW30, SW28 to SW31, SW29 to SW32, SW30 to SW33, SW31 to SW34, SW32 to SW35, SW33 to SW36, SW34 to SW37, SW35 to SW38, SW36 to SW39, SW55 to SW4, SW37 to SW40, SW38 to SW41, SW39 to SW42, SW40 to SW43, SW50 to SW44, SW41 to SW45, SW42 to SW46, SW43 to SW47, SW44 to SW48, SW60 to SW49, SW45 to SW5, SW46 to SW50, SW47 to SW51, SW48 to SW52, SW49 to SW53, SW64 to SW54, SW51 to SW55, SW52 to SW56, SW53 to SW57, SW54 to SW58, SW65 to SW59, SW2 to SW6, SW56 to SW60, SW57 to SW61, SW58 to SW62, SW59 to SW63, SW69 to SW64, SW61 to SW65, SW62 to SW67, SW67 to SW68, SW63 to SW69, SW3 to SW7, SW4 to SW8, SW5 to SW9
Connections:
- net C0: now also SW5.2 (B); no longer SW10.2 (B)
- net C1: now also SW10.2 (B); no longer SW15.2 (B)
- net C2: now also SW15.2 (B); no longer SW20.2 (B)
- net C3: now also SW20.2 (B); no longer SW25.2 (B)
- net C4: now also SW25.2 (B)
- net C5: no longer SW34.2 (B)
- net C6: now also SW34.2 (B); no longer SW39.2 (B)
- net C7: now also SW39.2 (B); no longer SW5.2 (B)
Other:
- moved on the sheet: D11, D16, D21, D26, D35, D40, D6, SW10, SW15, SW20, SW25, SW34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

Commit message: Use both types of joystick
Parts:
- removed D26, D40: D, Diode_THT:D_DO-35_SOD27_P7.62mm_Horizontal, symbol Device:D
- removed SW25: SW_m_left, Switch_Keyboard_Hotswap_Kailh:SW_Hotswap_Kailh_MX_1.00u, symbol Switch:SW_SPST
- removed SW39: SW_m_right, Switch_Keyboard_Hotswap_Kailh:SW_Hotswap_Kailh_MX_1.00u, symbol Switch:SW_SPST
Changed lines of the file:
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@@
   (junction (at 125.73 80.01) (diameter 0) (color 0 0 0 0)
   )
-  (junction (at 161.29 140.97) (diameter 0) (color 0 0 0 0)
-  )
   (junction (at 69.85 105.41) (diameter 0) (color 0 0 0 0)
   )
@@
   (junction (at 262.89 97.79) (diameter 0) (color 0 0 0 0)
   )
-  (junction (at 171.45 115.57) (diameter 0) (color 0 0 0 0)
-  )
   (junction (at 146.05 87.63) (diameter 0) (color 0 0 0 0)
   )
@@
   (junction (at 54.61 105.41) (diameter 0) (color 0 0 0 0)
   )
-  (junction (at 125.73 115.57) (diameter 0) (color 0 0 0 0)
-  )
   (junction (at 85.09 140.97) (diameter 0) (color 0 0 0 0)
   )
@@
   (junction (at 247.65 97.79) (diameter 0) (color 0 0 0 0)
   )
-  (junction (at 115.57 140.97) (diameter 0) (color 0 0 0 0)
-  )
   (junction (at 110.49 115.57) (diameter 0) (color 0 0 0 0)
   )
@@
     (stroke (width 0) (type default) (color 0 0 0 0))
   )
-  (wire (pts (xy 115.57 140.97) (xy 146.05 140.97))
-    (stroke (width 0) (type default) (color 0 0 0 0))
-  )
   (wire (pts (xy 176.53 87.63) (xy 191.77 87.63))
     (stroke (width 0) (type default) (color 0 0 0 0))
@@
     (stroke (width 0) (type default) (color 0 0 0 0))
   )
-  (wire (pts (xy 171.45 115.57) (xy 171.45 133.35))
-    (stroke (width 0) (type default) (color 0 0 0 0))
-  )
   (wire (pts (xy 110.49 62.23) (xy 110.49 80.01))
     (stroke (width 0) (type default) (color 0 0 0 0))
@@
     (stroke (width 0) (type default) (color 0 0 0 0))
   )
-  (wire (pts (xy 161.29 140.97) (xy 176.53 140.97))
+  (wire (pts (xy 146.05 140.97) (xy 176.53 140.97))
     (stroke (width 0) (type default) (color 0 0 0 0))
   )
@@
     (stroke (width 0) (type default) (color 0 0 0 0))
   )
-  (wire (pts (xy 146.05 140.97) (xy 161.29 140.97))
-    (stroke (width 0) (type default) (color 0 0 0 0))
-  )
   (wire (pts (xy 222.25 69.85) (xy 237.49 69.85))
     (stroke (width 0) (type default) (color 0 0 0 0))
@@
     (stroke (width 0) (type default) (color 0 0 0 0))
   )
-  (wire (pts (xy 125.73 115.57) (xy 125.73 133.35))
-    (stroke (width 0) (type default) (color 0 0 0 0))
-  )
   (wire (pts (xy 146.05 105.41) (xy 161.29 105.41))
     (stroke (width 0) (type default) (color 0 0 0 0))
@@
     (stroke (width 0) (type default) (color 0 0 0 0))
   )
-  (wire (pts (xy 100.33 140.97) (xy 115.57 140.97))
+  (wire (pts (xy 100.33 140.97) (xy 146.05 140.97))
     (stroke (width 0) (type default) (color 0 0 0 0))
   )
@@
     (pin "2")
   )
-  (symbol (lib_id "Device:D") (at 115.57 137.16 90) (unit 1)
-    (in_bom yes) (on_board yes) (fields_autoplaced)
-    (property "Reference" "D26" (id 0) (at 118.11 135.8899 90)
-      (effects (font (size 1.27 1.27)) (justify right))
-    )
-    (property "Value" "D" (id 1) (at 118.11 138.4299 90)
-      (effects (font (size 1.27 1.27)) (justify right))
-    )
-    (property "Footprint" "Diode_THT:D_DO-35_SOD27_P7.62mm_Horizontal" (id 2) (at 115.57 137.16 0)
-      (effects (font (size 1.27 1.27)) hide)
-    )
-    (property "Datasheet" "~" (id 3) (at 115.57 137.16 0)
-      (effects (font (size 1.27 1.27)) hide)
-    )
-    (pin "1")
-    (pin "2")
-  )
   (symbol (lib_id "Device:D") (at 207.01 83.82 90) (unit 1)
     (in_bom yes) (on_board yes) (fields_autoplaced)
@@
     (pin "2")
   )
-  (symbol (lib_id "Switch:SW_SPST") (at 166.37 133.35 0) (unit 1)
-    (in_bom yes) (on_board yes) (fields_autoplaced)
-    (property "Reference" "SW39" (id 0) (at 166.37 127 0))
-    (property "Value" "SW_m_right" (id 1) (at 166.37 129.54 0))
-    (property "Footprint" "Switch_Keyboard_Hotswap_Kailh:SW_Hotswap_Kailh_MX_1.00u" (id 2) (at 166.37 133.35 0)
-      (effects (font (size 1.27 1.27)) hide)
-    )
-    (property "Datasheet" "~" (id 3) (at 166.37 133.35 0)
-      (effects (font (size 1.27 1.27)) hide)
-    )
-    (pin "1")
-    (pin "2")
-  )
   (symbol (lib_id "Device:D") (at 85.09 66.04 90) (unit 1)
     (in_bom yes) (on_board yes) (fields_autoplaced)
@@
     (pin "2")
   )
-  (symbol (lib_id "Switch:SW_SPST") (at 120.65 133.35 0) (unit 1)
-    (in_bom yes) (on_board yes) (fields_autoplaced)
-    (property "Reference" "SW25" (id 0) (at 120.65 127 0))
-    (property "Value" "SW_m_left" (id 1) (at 120.65 129.54 0))
-    (property "Footprint" "Switch_Keyboard_Hotswap_Kailh:SW_Hotswap_Kailh_MX_1.00u" (id 2) (at 120.65 133.35 0)
-      (effects (font (size 1.27 1.27)) hide)
-    )
-    (property "Datasheet" "~" (id 3) (at 120.65 133.35 0)
-      (effects (font (size 1.27 1.27)) hide)
-    )
-    (pin "1")
-    (pin "2")
-  )
   (symbol (lib_id "Device:D") (at 146.05 119.38 90) (unit 1)
     (in_bom yes) (on_board yes) (fields_autoplaced)
@@
       (effects (font (size 1.27 1.27)) hide)
     )
-    (pin "1")
-    (pin "2")
-  )
-  (symbol (lib_id "Device:D") (at 161.29 137.16 90) (unit 1)
-    (in_bom yes) (on_board yes) (fields_autoplaced)
-    (property "Reference" "D40" (id 0) (at 163.83 135.8899 90)
-      (effects (font (size 1.27 1.27)) (justify right))
-    )
-    (property "Value" "D" (id 1) (at 163.83 138.4299 90)
-      (effects (font (size 1.27 1.27)) (justify right))
-    )
-    (property "Footprint" "Diode_THT:D_DO-35_SOD27_P7.62mm_Horizontal" (id 2) (at 161.29 137.16 0)
-      (effects (font (size 1.27 1.27)) hide)
-    )
-    (property "Datasheet" "~" (id 3) (at 161.29 137.16 0)
-      (effects (font (size 1.27 1.27)) hide)
-    )
